File: pcb/2102_sram_tester.kicad_pcb (KiCad board)
At the start: 2 copper layers, 63.5 x 61 mm, 11 parts, among them SW1 SW_Push

Commit message: Added firmware and updated PCB
Connections:
- A1 pad 19: Net-(A1-A0) -> unconnected-(A1-A0-Pad19)
- A1 pad 25: D_{out} -> unconnected-(A1-A6-Pad25)
- A1 pad 5: unconnected-(A1-D2-Pad5) -> Net-(A1-D2)
- A1 pad 6: unconnected-(A1-D3-Pad6) -> D_{out}
- SW1 pad 1: Net-(A1-A0) -> GND
- SW1 pad 2: GND -> Net-(A1-D2)
Routing:
- net Net-(A1-D2): track 0.00 -> 75.4 mm
- net D_{out}: track 27.4 -> 68.4 mm
- net Net-(A1-A0): track 23.1 -> 0.00 mm
- net A3: track 49.7 -> 47.8 mm
- net ~{CS}: track 36.5 -> 34.9 mm
- net A4: track 49.0 -> 47.6 mm
