File: pcb/2102_sram_tester.kicad_sch (KiCad schematic)
At the start: 11 parts, among them SW1 SW_Push

Commit message: Added firmware and updated PCB
Connections:
- net D_{out}: now also A1.6 (D3); no longer A1.25 (A6)
- net GND: now also SW1.1; no longer SW1.2
- net at A1.19 (A0): no longer SW1.1
- net at A1.5 (D2): now also SW1.2
Other:
- note added: "Note: Input Only"
- moved on the sheet: D1, D2, H1, H2, H3, H4, R1, R2, SW1, U1
